Commit message: - added plotting - added library scenario

File: panda_gym/assets/scenarios/library/shelf.urdf (robot description, URDF)
Before this commit: robot shelf, 1 links, 0 joints
Links:
- link shelf_base_link: geometry collision mesh filename=shelf.obj scale=0.0008 0.0008 0.0008; visual mesh filename=shelf.obj scale=0.0008 0.0008 0.0008

File: panda_gym/assets/scenarios/library/table.urdf (robot description, URDF)
Before this commit: robot table, 1 links, 0 joints
Links:
- link table_base_link: geometry collision mesh filename=table.obj scale=0.0008 0.0008 0.0008; visual mesh filename=table.obj scale=0.0008 0.0008 0.0008

Commit message: - reach evade obstacle changes

File: panda_gym/assets/scenarios/library/shelf.urdf (robot description, URDF)
Before this commit: robot shelf, 1 links, 0 joints
Links:
- link shelf_base_link: geometry collision mesh filename=shelf.obj scale=0.0009 0.0009 0.0009; visual mesh filename=shelf.obj scale=0.0009 0.0009 0.0009
