Commit message: - udpatesd

File: panda_gym/URDF/robots/franka_panda_custom/panda.urdf (robot description, URDF)
Before this commit: robot panda, 13 links, 12 joints
Links:
- link panda_link8: geometry collision cylinder length=0.01 radius=0.03; collision sphere radius=0.03
Joints:
- joint panda_finger_joint1: type prismatic -> fixed
- joint panda_finger_joint2: type prismatic -> fixed
