Commit message: - many changes

File: panda_gym/assets/scenarios/workshop/urdf/box1.urdf (robot description, URDF)
Before this commit: robot box1, 1 links, 0 joints
Links:
- link box1_base_link: geometry collision mesh filename=../meshes/box1.obj scale=0.0005 0.0005 0.0005; visual mesh filename=../meshes/box1.obj scale=0.0005 0.0005 0.0005

File: panda_gym/assets/scenarios/workshop/urdf/box2.urdf (robot description, URDF)
Before this commit: robot box2, 1 links, 0 joints
Links:
- link box2_base_link: geometry collision mesh filename=../meshes/box2.obj scale=0.0005 0.0005 0.0005; visual mesh filename=../meshes/box2.obj scale=0.0005 0.0005 0.0005

File: panda_gym/assets/scenarios/workshop/urdf/box3.urdf (robot description, URDF)
Before this commit: robot box3, 1 links, 0 joints
Links:
- link box3_base_link: geometry collision mesh filename=../meshes/box3.obj scale=0.0005 0.0005 0.0005; visual mesh filename=../meshes/box3.obj scale=0.0005 0.0005 0.0005

File: panda_gym/assets/scenarios/workshop/urdf/part_box.urdf (robot description, URDF)
Before this commit: robot part_box, 1 links, 0 joints
Links:
- link part_box_base_link: geometry collision mesh filename=../meshes/part_box.obj scale=0.0005 0.0005 0.0005; visual mesh filename=../meshes/part_box.obj scale=0.0005 0.0005 0.0005

File: panda_gym/assets/scenarios/workshop/urdf/table1.urdf (robot description, URDF)
Before this commit: robot table1, 1 links, 0 joints
Links:
- link table1_base_link: geometry collision mesh filename=../meshes/table1.obj scale=0.0005 0.0005 0.0005; visual mesh filename=../meshes/table1.obj scale=0.0005 0.0005 0.0005

File: panda_gym/assets/scenarios/workshop/urdf/table2.urdf (robot description, URDF)
Before this commit: robot table2, 1 links, 0 joints
Links:
- link table2_base_link: geometry collision mesh filename=../meshes/table2.obj scale=0.0005 0.0005 0.0005; visual mesh filename=../meshes/table2.obj scale=0.0005 0.0005 0.0005
