Commit message: - small changes, additions and bug fixes

File: panda_gym/assets/robots/franka_panda_custom/panda.urdf (robot description, URDF)
Before this commit: robot panda, 13 links, 12 joints
Links:
- added link panda_hand_collision_1, mass 1e-6; collision cylinder length=0.1 radius=0.04; visual sphere radius=0.0001
- added link panda_hand_collision_2, mass 1e-6; collision sphere radius=0.04; visual box size=0.0001 0.0001 0.0001
- added link panda_hand_collision_3, mass 1e-6; collision sphere radius=0.04; visual cylinder length=0.0001 radius=0.0001
- added link panda_hand_collision_4, mass 1e-6; collision cylinder length=0.1 radius=0.02; visual sphere radius=0.0001
- added link panda_hand_collision_5, mass 1e-6; collision sphere radius=0.02; visual box size=0.0001 0.0001 0.0001
- added link panda_hand_collision_6, mass 1e-6; collision sphere radius=0.02; visual cylinder length=0.0001 radius=0.0001
- link panda_hand: geometry visual mesh filename=package://meshes/visual/hand.obj
Joints:
- added joint panda_hand_collision_1_joint: type fixed, parent panda_hand, child panda_hand_collision_1, origin xyz=0 0 0 rpy=0 0 0
- added joint panda_hand_collision_2_joint: type fixed, parent panda_hand, child panda_hand_collision_2, origin xyz=0 0 0 rpy=0 0 0
- added joint panda_hand_collision_3_joint: type fixed, parent panda_hand, child panda_hand_collision_3, origin xyz=0 0 0 rpy=0 0 0
- added joint panda_hand_collision_4_joint: type fixed, parent panda_hand, child panda_hand_collision_4, origin xyz=0 0 0 rpy=0 0 0
- added joint panda_hand_collision_5_joint: type fixed, parent panda_hand, child panda_hand_collision_5, origin xyz=0 0 0 rpy=0 0 0
- added joint panda_hand_collision_6_joint: type fixed, parent panda_hand, child panda_hand_collision_6, origin xyz=0 0 0 rpy=0 0 0

File: panda_gym/assets/scenarios/tabletop/urdf/tabletop.urdf (robot description, URDF)
Before this commit: robot tabletop, 2 links, 1 joints
Links:
- removed link tabletop
- added link back_wall; collision box size=0.01 1.2 1.0; visual box size=0.01 1.2 1.0
- added link cabinet_bottom; collision box size=0.2 0.835 0.01; visual box size=0.2 0.835 0.01
- added link cabinet_left_wall; collision box size=0.2 0.01 0.35; visual box size=0.2 0.01 0.35
- added link cabinet_middle_wall; collision box size=0.2 0.01 0.35; visual box size=0.2 0.01 0.35
- added link cabinet_right_wall; collision box size=0.2 0.01 0.35; visual box size=0.2 0.01 0.35
- added link cabinet_shelf; collision box size=0.2 0.835 0.01; visual box size=0.2 0.835 0.01
- added link cabinet_top; collision box size=0.2 0.835 0.01; visual box size=0.2 0.835 0.01
- added link cold_water_knob; collision box size=0.015 0.015 0.03; visual box size=0.015 0.015 0.03
- added link countertop_left; collision box size=0.3 0.3 0.01; visual box size=0.3 0.3 0.01
- added link countertop_right; collision box size=0.3 0.26 0.01; visual box size=0.3 0.26 0.01
- added link dishwasher_back_wall; collision box size=0.01 0.24 0.37; visual box size=0.01 0.24 0.37
- added link dishwasher_bottom; collision box size=0.28 0.24 0.01; visual box size=0.28 0.24 0.01
- added link dishwasher_bottom_wall; collision box size=0.01 0.24 0.08; visual box size=0.01 0.24 0.08
- added link dishwasher_door; collision box size=0.3 0.24 0.01; visual box size=0.3 0.24 0.01
- added link dishwasher_front_top_wall; collision box size=0.01 0.24 0.04; visual box size=0.01 0.24 0.04
- added link dishwasher_handle; collision box size=0.015 0.165 0.015; visual box size=0.015 0.165 0.015
- added link dishwasher_handle_left; collision box size=0.015 0.015 0.035; visual box size=0.015 0.015 0.035
- added link dishwasher_handle_right; collision box size=0.015 0.015 0.035; visual box size=0.015 0.015 0.035
- added link dishwasher_left_side; collision box size=0.3 0.01 0.375; visual box size=0.3 0.01 0.375
- added link dishwasher_right_side; collision box size=0.3 0.01 0.375; visual box size=0.3 0.01 0.375
- added link faucet_1; collision box size=0.015 0.015 0.15; visual box size=0.015 0.015 0.15
- added link faucet_2; collision box size=0.125 0.015 0.015; visual box size=0.125 0.015 0.015
- added link faucet_3; collision box size=0.01 0.01 0.025; visual box size=0.01 0.01 0.025
- added link faucet_platform; collision box size=0.04 0.3 0.01; visual box size=0.04 0.3 0.01
- added link freezer_door; collision box size=0.01 0.35 0.3; visual box size=0.01 0.35 0.3
- added link freezer_handle; collision box size=0.015 0.15 0.015; visual box size=0.015 0.15 0.015
- added link freezer_handle_left; collision box size=0.035 0.015 0.015; visual box size=0.035 0.015 0.015
- added link freezer_handle_right; collision box size=0.035 0.015 0.015; visual box size=0.035 0.015 0.015
- added link fridge_back_wall; collision box size=0.01 0.35 0.75; visual box size=0.01 0.35 0.75
- added link fridge_door; collision box size=0.35 0.01 0.45; visual box size=0.35 0.01 0.45
- added link fridge_left_wall; collision box size=0.3 0.01 0.75; visual box size=0.3 0.01 0.75
- added link fridge_right_wall; collision box size=0.3 0.01 0.75; visual box size=0.3 0.01 0.75
- added link fridge_shelf1; collision box size=0.295 0.35 0.01; visual box size=0.295 0.35 0.01
- added link fridge_shelf2; collision box size=0.295 0.35 0.01; visual box size=0.295 0.35 0.01
- added link fridge_shelf3; collision box size=0.295 0.35 0.01; visual box size=0.295 0.35 0.01
- added link fridge_top; collision box size=0.3 0.355 0.01; visual box size=0.3 0.355 0.01
- added link hot_water_knob; collision box size=0.015 0.015 0.03; visual box size=0.015 0.015 0.03
- added link lower_cabinet_back_wall; collision box size=0.01 0.3 0.375; visual box size=0.01 0.3 0.375
- added link lower_cabinet_bottom; collision box size=0.3 0.3 0.01; visual box size=0.3 0.3 0.01
- added link lower_cabinet_left_wall; collision box size=0.3 0.01 0.38; visual box size=0.3 0.01 0.38
- added link lower_cabinet_right_wall; collision box size=0.3 0.01 0.38; visual box size=0.3 0.01 0.38
- added link lower_cabinet_shelf; collision box size=0.3 0.3 0.01; visual box size=0.3 0.3 0.01
- added link sink_back_wall; collision box size=0.01 0.31 0.38; visual box size=0.01 0.31 0.38
- added link sink_bottom; collision box size=0.3 0.3 0.01; visual box size=0.3 0.3 0.01
- added link sink_front_wall; collision box size=0.01 0.32 0.38; visual box size=0.01 0.32 0.38
- added link sink_left_wall; collision box size=0.3 0.01 0.125; visual box size=0.3 0.01 0.125
- added link sink_right_wall; collision box size=0.3 0.01 0.125; visual box size=0.3 0.01 0.125
Joints:
- removed joint tabletop_joint
- added joint back_wall_joint: type fixed, parent world, child back_wall, origin xyz=0.0025 0.3 0.25 rpy=0 0 0
- added joint cabinet_bottom_joint: type fixed, parent world, child cabinet_bottom, origin xyz=0.05 0.39125 0.3 rpy=0 0 0
- added joint cabinet_left_wall_joint: type fixed, parent world, child cabinet_left_wall, origin xyz=0.05 0.185 0.3875 rpy=0 0 0
- added joint cabinet_middle_wall_joint: type fixed, parent world, child cabinet_middle_wall, origin xyz=0.05 0.405 0.3875 rpy=0 0 0
- added joint cabinet_right_wall_joint: type fixed, parent world, child cabinet_right_wall, origin xyz=0.05 0.5975 0.3875 rpy=0 0 0
- added joint cabinet_shelf_joint: type fixed, parent world, child cabinet_shelf, origin xyz=0.05 0.39125 0.3875 rpy=0 0 0
- added joint cabinet_top_joint: type fixed, parent world, child cabinet_top, origin xyz=0.05 0.39125 0.475 rpy=0 0 0
- added joint cold_water_knob_joint: type fixed, parent world, child cold_water_knob, origin xyz=0.01 0.375 0.195 rpy=0 0 0
- added joint countertop_left_joint: type fixed, parent world, child countertop_left, origin xyz=0.075 0.2525 0.1875 rpy=0 0 0
- added joint countertop_right_joint: type fixed, parent world, child countertop_right, origin xyz=0.075 0.535 0.1875 rpy=0 0 0
- added joint dishwasher_back_wall_joint: type fixed, parent world, child dishwasher_back_wall, origin xyz=0.005 0.5375 0.0875 rpy=0 0 0
- added joint dishwasher_bottom_joint: type fixed, parent world, child dishwasher_bottom, origin xyz=0.075 0.5375 0.025 rpy=0 0 0
- added joint dishwasher_bottom_wall_joint: type fixed, parent world, child dishwasher_bottom_wall, origin xyz=0.15 0.54 0.02 rpy=0 0 0
- added joint dishwasher_door_joint: type fixed, parent world, child dishwasher_door, origin xyz=0.225 0.54 0.04 rpy=0 0 0
- added joint dishwasher_front_top_wall_joint: type fixed, parent world, child dishwasher_front_top_wall, origin xyz=0.1525 0.54 0.18 rpy=0 0 0
- added joint dishwasher_handle_joint: type fixed, parent world, child dishwasher_handle, origin xyz=0.275 0.5375 0.02 rpy=0 0 0
- added joint dishwasher_handle_left_joint: type fixed, parent world, child dishwasher_handle_left, origin xyz=0.275 0.5 0.03 rpy=0 0 0
- added joint dishwasher_handle_right_joint: type fixed, parent world, child dishwasher_handle_right, origin xyz=0.275 0.575 0.03 rpy=0 0 0
- added joint dishwasher_left_side_joint: type fixed, parent world, child dishwasher_left_side, origin xyz=0.075 0.4775 0.09375 rpy=0 0 0
- added joint dishwasher_right_side_joint: type fixed, parent world, child dishwasher_right_side, origin xyz=0.075 0.5975 0.09375 rpy=0 0 0
- added joint faucet_1_joint: type fixed, parent world, child faucet_1, origin xyz=0.01 0.4 0.225 rpy=0 0 0
- added joint faucet_2_joint: type fixed, parent world, child faucet_2, origin xyz=0.0375 0.4 0.2625 rpy=0 0 0
- added joint faucet_3_joint: type fixed, parent world, child faucet_3, origin xyz=0.06625 0.4 0.25625 rpy=0 0 0
- added joint faucet_platform_joint: type fixed, parent world, child faucet_platform, origin xyz=0.01 0.4 0.1875 rpy=0 0 0
- added joint freezer_door_joint: type fixed, parent world, child freezer_door, origin xyz=0.15 0.0875 0.075 rpy=0 0 0
- added joint freezer_handle_joint: type fixed, parent world, child freezer_handle, origin xyz=0.1625 0.0875 0.1375 rpy=0 0 0
- added joint freezer_handle_left_joint: type fixed, parent world, child freezer_handle_left, origin xyz=0.1575 0.05 0.1375 rpy=0 0 0
- added joint freezer_handle_right_joint: type fixed, parent world, child freezer_handle_right, origin xyz=0.1575 0.125 0.1375 rpy=0 0 0
- added joint fridge_back_wall_joint: type fixed, parent world, child fridge_back_wall, origin xyz=0.005 0.0875 0.1875 rpy=0 0 0
- added joint fridge_door_joint: type fixed, parent world, child fridge_door, origin xyz=0.1625 0.0025 0.265 rpy=0 0 0
- added joint fridge_left_wall_joint: type fixed, parent world, child fridge_left_wall, origin xyz=0.075 0.0025 0.1875 rpy=0 0 0
- added joint fridge_right_wall_joint: type fixed, parent world, child fridge_right_wall, origin xyz=0.075 0.175 0.1875 rpy=0 0 0
- added joint fridge_shelf1_joint: type fixed, parent world, child fridge_shelf1, origin xyz=0.075 0.0875 0.3075 rpy=0 0 0
- added joint fridge_shelf2_joint: type fixed, parent world, child fridge_shelf2, origin xyz=0.075 0.0875 0.23 rpy=0 0 0
- added joint fridge_shelf3_joint: type fixed, parent world, child fridge_shelf3, origin xyz=0.075 0.0875 0.15 rpy=0 0 0
- added joint fridge_top_joint: type fixed, parent world, child fridge_top, origin xyz=0.075 0.08875 0.375 rpy=0 0 0
- added joint hot_water_knob_joint: type fixed, parent world, child hot_water_knob, origin xyz=0.01 0.425 0.195 rpy=0 0 0
- added joint lower_cabinet_back_wall_joint: type fixed, parent world, child lower_cabinet_back_wall, origin xyz=0.005 0.25 0.0925 rpy=0 0 0
- added joint lower_cabinet_bottom_joint: type fixed, parent world, child lower_cabinet_bottom, origin xyz=0.075 0.25 0.0025 rpy=0 0 0
- added joint lower_cabinet_left_wall_joint: type fixed, parent world, child lower_cabinet_left_wall, origin xyz=0.075 0.18 0.095 rpy=0 0 0
- added joint lower_cabinet_right_wall_joint: type fixed, parent world, child lower_cabinet_right_wall, origin xyz=0.075 0.3225 0.095 rpy=0 0 0
- added joint lower_cabinet_shelf_joint: type fixed, parent world, child lower_cabinet_shelf, origin xyz=0.075 0.25 0.0875 rpy=0 0 0
- added joint sink_back_wall_joint: type fixed, parent world, child sink_back_wall, origin xyz=0.0075 0.4 0.095 rpy=0 0 0
- added joint sink_bottom_joint: type fixed, parent world, child sink_bottom, origin xyz=0.075 0.4 0.125 rpy=0 0 0
- added joint sink_front_wall_joint: type fixed, parent world, child sink_front_wall, origin xyz=0.15 0.4 0.095 rpy=0 0 0
- added joint sink_left_wall_joint: type fixed, parent world, child sink_left_wall, origin xyz=0.075 0.325 0.15625 rpy=0 0 0
- added joint sink_right_wall_joint: type fixed, parent world, child sink_right_wall, origin xyz=0.075 0.475 0.15625 rpy=0 0 0
